Commit message: doc: adding robot localization

File: src/my_robot_description/urdf/common_properties.xacro (robot description, xacro)
@@ -6,4 +6,7 @@
     <material name="grey">
         <color rgba="0.5 0.5 0.5 1" />
+    </material>
+    <material name="orange">
+    <color rgba="${255/255} ${108/255} ${10/255} 1.0"/>
     </material>
     <xacro:macro name="box_inertia" params="m l w h xyz rpy">

File: src/my_robot_description/urdf/mobile_base_gazebo.xacro (robot description, xacro)
@@ -18,4 +18,7 @@
     <gazebo>
         <plugin name="diff_drive_controller" filename="libgazebo_ros_diff_drive.so">
+            <!-- <ros>
+                <namespace>/demo</namespace>
+            </ros> -->
             <!-- Update rate in Hz -->
             <update_rate>50</update_rate>
@@ -29,6 +32,6 @@
             <command_topic>cmd_vel</command_topic>
             <!-- output pub -->
-            <publish_odom>true</publish_odom> <!-- where the robot compere to the origin(starting point)-->
-            <publish_odom_tf>true</publish_odom_tf>
+            <publish_odom>true</publish_odom>
+            <publish_odom_tf>false</publish_odom_tf>
             <publish_wheel_tf>true</publish_wheel_tf>
             <odometry_topic>odom</odometry_topic>

File: src/my_robot_description/urdf/my_robot.urdf.xacro (robot description, xacro)
@@ -4,3 +4,4 @@
     <xacro:include filename="mobile_base.xacro" />
     <xacro:include filename="mobile_base_gazebo.xacro" />
+    <xacro:include filename="base_scan.xacro" />
 </robot>
