Commit message: doc:adding map with slam toolbox

File: src/my_robot_description/urdf/base_scan.xacro (robot description, xacro)
@@ -1,5 +1,5 @@
 <?xml version="1.0"?>
 <robot name="my_robot" xmlns:xacro="http://www.ros.org/wiki/xacro">
-    <xacro:arg name="laser_visual"  default="true"/>
+    <xacro:arg name="laser_visual"  default="false"/>
     <xacro:property name ="scan_radius" value="0.1" />
     <xacro:property name ="scan_length" value="0.06" />

File: src/my_robot_description/urdf/camera.xacro (robot description, xacro)
@@ -24,7 +24,13 @@
         <origin xyz="${(base_length + camera_length) / 2.0 } 0 ${base_height / 2.0}" rpy="0 0 0" />
     </joint>
+    <joint name="camera_optical_joint" type="fixed">
+        <parent link="camera_link" />
+        <child link="camera_link_optical" />
+        <origin xyz="0 0 0" rpy="${-pi/2} 0 ${-pi/2}" />
+    </joint>
+    <link name="camera_link_optical"></link>
     <gazebo reference="camera_link">
         <material>Gazebo/Red</material>
-        <sensor name="depth_camera" type="depth">
+        <sensor name="camera" type="depth">
                 <pose>0 0 0 0 0 0 </pose>
                 <visualize>true</visualize>
@@ -35,5 +41,5 @@
                         <width>640</width>
                         <height>480</height>
-                        <format>R8G8B8</format>
+                        <format>B8G8R8</format>
                     </image>
                     <clip>
@@ -46,17 +52,7 @@
                     <alwaysOn>true</alwaysOn>
                     <updateRate>0.0</updateRate>
-                    <frame_name>camera_link</frame_name>
-                    <pointCloudCutoff>0.5</pointCloudCutoff>
-                    <pointCloudCutoffMax>3.0</pointCloudCutoffMax>
-                    <distortionK1>0</distortionK1>
-                    <distortionK2>0</distortionK2>
-                    <distortionK3>0</distortionK3>
-                    <distortionT1>0</distortionT1>
-                    <distortionT2>0</distortionT2>
-                    <CxPrime>0</CxPrime>
-                    <Cx>0</Cx>
-                    <Cy>0</Cy>
-                    <focalLength>0</focalLength>
-                    <hackBaseline>0</hackBaseline>
+                    <frame_name>camera_link_optical</frame_name>
+                    <min_depth>0.1</min_depth>
+                    <max_depth>100</max_depth>
                 </plugin>
         </sensor>

File: src/my_robot_description/urdf/mobile_base.xacro (robot description, xacro)
@@ -63,6 +63,6 @@
     </link>
     <joint name="base_joint" type="fixed">
-        <parent link="base_footprint" />
-        <child link="base_link" />
+        <parent link="base_link"/>
+        <child link="base_footprint"/>
         <origin xyz="0 0 ${wheel_radius}" rpy="0 0 0"/>
     </joint>

File: src/my_robot_description/urdf/mobile_base_gazebo.xacro (robot description, xacro)
@@ -11,16 +11,16 @@
     </gazebo>
     <gazebo reference="caster_wheel_link">
-        <material>Gazebo/Grey</material>
-        <mu1 value="0.1" />
-        <mu2 value="0.1" />
+        <material>Gazebo/Black</material>
+        <mu1 value="0.001" />
+        <mu2 value="0.001" />
     </gazebo>
         <!-- Install gazebo_ros_pkgs sudo apt install ros-humble-gazebo-ros-pkgs -->
     <gazebo>
-        <plugin name="diff_drive_controller" filename="libgazebo_ros_diff_drive.so">
+        <plugin name="diff_drive" filename="libgazebo_ros_diff_drive.so">
             <!-- <ros>
-                <namespace>/demo</namespace>
+                <namespace>/pub</namespace>
             </ros> -->
             <!-- Update rate in Hz -->
-            <update_rate>50</update_rate>
+            <update_rate>30</update_rate>
             <!-- wheels -->
             <left_joint>base_left_wheel_joint</left_joint> <!--name of the joint-->
@@ -29,13 +29,15 @@
             <wheel_separation>0.45</wheel_separation> <!-- distance between the wheels, base+half the wheel length-->
             <wheel_diameter>0.2</wheel_diameter> <!--2*wheel radius-->
+            <!-- Limits -->
+            <max_wheel_torque>200</max_wheel_torque>
+            <max_wheel_acceleration>10.0</max_wheel_acceleration>
             <!-- input -->
             <command_topic>cmd_vel</command_topic>
-            <!-- output pub -->
+            <!-- Output -->
+            <odometry_frame>odom</odometry_frame>
+            <robot_base_frame>base_link</robot_base_frame> <!--base view point-->
             <publish_odom>true</publish_odom>
-            <publish_odom_tf>false</publish_odom_tf>
+            <publish_odom_tf>true</publish_odom_tf>
             <publish_wheel_tf>true</publish_wheel_tf>
-            <odometry_topic>odom</odometry_topic>
-            <odometry_frame>odom</odometry_frame>
-            <robot_base_frame>base_footprint</robot_base_frame> <!--base view point-->
         </plugin>
     </gazebo>
